File: PCB/Heptachron/Heptachron.kicad_pcb (KiCad board)
At the start: 2 copper layers, 42 x 25 mm, 48 parts, among them IC1 BQ25185DLHR, J2 Conn_01x01_Pin, Q1 Q_Photo_NPN, SW1 SW_Push, SW2 SW_Push, SW4 SW_SP3T, U6 BQ24230RGT, U7 IS31FL3729, U8 ATtiny424-SS, X1 RV-3028-C7

Commit message: Continue PCB
Parts:
- removed C2, C3, C5: 4.7u, Capacitor_SMD:C_0805_2012Metric
- removed D1: PGD, LED_SMD:LED_0603_1608Metric
- removed D2: CHG, LED_SMD:LED_0603_1608Metric
- removed D3: BAT, LED_SMD:LED_0603_1608Metric
- removed D4: VCC, LED_SMD:LED_0603_1608Metric
- removed R10, R11, R12, R9: 1K, Resistor_SMD:R_0603_1608Metric
- removed R3, R4, R8: 10K, Resistor_SMD:R_0603_1608Metric
- removed R5: 3.3K, Resistor_SMD:R_0603_1608Metric
- removed R6: 4.7K, Resistor_SMD:R_0603_1608Metric
- removed R7: DNP, Resistor_SMD:R_0603_1608Metric
- removed SW4: SW_SP3T, Heptachron-Lib:sp3t_jumpers
- removed U6: BQ24230RGT, Package_DFN_QFN:VQFN-16-1EP_3x3mm_P0.5mm_EP1.68x1.68mm_ThermalVias
- added C10: 1u, Capacitor_SMD:C_0805_2012Metric, B.Cu at (152.5, 92.2)
- added C8: 1u, Capacitor_SMD:C_0805_2012Metric, B.Cu at (143.8, 89.9)
- added C9: 10u, Capacitor_SMD:C_0805_2012Metric, B.Cu at (152.5, 89.9)
- added D43: ~, LED_SMD:LED_0603_1608Metric, F.Cu at (153.0, 107.2)
- added J1: 5V, Connector_Wire:SolderWirePad_1x01_SMD_1x2mm, B.Cu at (159.4, 110.0)
- added J3: UPDI, Connector_Wire:SolderWirePad_1x01_SMD_1x2mm, B.Cu at (159.4, 108.5)
- added J4: BAT+, Connector_Wire:SolderWirePad_1x01_SMD_1x2mm, B.Cu at (136.6, 89.6)
- added J5: BAT-, Connector_Wire:SolderWirePad_1x01_SMD_1x2mm, B.Cu at (136.6, 91.3)
- added R17: 18K, Resistor_SMD:R_0603_1608Metric, B.Cu at (144.0, 93.7)
- added R18: 2K, Resistor_SMD:R_0603_1608Metric, B.Cu at (144.0, 91.9)
- added R19: 10K, Resistor_SMD:R_0603_1608Metric, B.Cu at (148.0, 93.6)
- added TP1: STAT1, TestPoint:TestPoint_Pad_D1.0mm, F.Cu at (96.0, 84.0)
- added TP2: STAT2, TestPoint:TestPoint_Pad_D1.0mm, F.Cu at (96.0, 90.1)
- added TP3: +5V, TestPoint:TestPoint_Pad_D1.0mm, F.Cu at (99.1, 84.0)
- added TP4: VCC, TestPoint:TestPoint_Pad_D1.0mm, F.Cu at (99.1, 90.1)
- added TP5: BAT, TestPoint:TestPoint_Pad_D1.0mm, F.Cu at (102.1, 84.0)
- added TP6: GND, TestPoint:TestPoint_Pad_D1.0mm, F.Cu at (102.1, 90.1)
- IC1: moved to B.Cu
- J2: value Conn_01x01_Pin -> GND; moved to B.Cu
- Q1: value Q_Photo_NPN -> Q_PH
- moved J2 48.8 mm to (159.4, 111.5), turned to 90 degrees
- moved Q1 37.0 mm to (148.0, 89.8)
- moved IC1 20.2 mm to (148.0, 91.2), turned to 180 degrees
- moved C7 17.0 mm to (172.5, 119.0)
- moved R15 17.0 mm to (173.0, 121.5)
- moved D38 1.00 mm to (151.0, 107.2)
- moved D39 1.00 mm to (149.0, 107.2)
- moved D40 1.00 mm to (147.0, 107.2)
- moved D41 1.00 mm to (145.0, 107.2)
- moved D42 1.00 mm to (143.0, 107.2)
- moved U8 0.25 mm to (164.8, 101.0)
Connections:
- IC1 pad 1: unconnected-(IC1-SYS-Pad1) -> VCC
- IC1 pad 10: unconnected-(IC1-IN-Pad10) -> +5V
- IC1 pad 11: unconnected-(IC1-EP-Pad11) -> GND
- IC1 pad 2: unconnected-(IC1-BAT-Pad2) -> +BATT
- IC1 pad 3: unconnected-(IC1-STAT2-Pad3) -> /STAT2
- IC1 pad 4: unconnected-(IC1-~{CE}-Pad4) -> //CE
- IC1 pad 5: unconnected-(IC1-GND-Pad5) -> GND
- IC1 pad 6: unconnected-(IC1-TS/MR-Pad6) -> Net-(IC1-TS/MR)
- IC1 pad 7: unconnected-(IC1-ILIM/VSET-Pad7) -> Net-(IC1-ILIM/VSET)
- IC1 pad 8: unconnected-(IC1-ISET-Pad8) -> Net-(IC1-ISET)
- IC1 pad 9: unconnected-(IC1-STAT1-Pad9) -> /STAT1
- J2 pad 1: unconnected-(J2-Pin_1-Pad1) -> GND
- U8 pad 11: /TX -> unconnected-(U8-PA1-Pad11)
- U8 pad 12: /RX -> unconnected-(U8-PA2-Pad12)
- U8 pad 3: /PGOOD -> /RTC_INT
- X1 pad 2: unconnected-(X1-INT-Pad2) -> /RTC_INT
Other:
- board text added: "BQ25185DLHR"
- board text removed: "TEST BOARD, NOT FUNCTIONAL"

Commit message: Continue PCB
Parts:
- removed TP3: +5V, TestPoint:TestPoint_Pad_D1.0mm
- removed TP5: BAT, TestPoint:TestPoint_Pad_D1.0mm
- added H1: MountingHole, Heptachron-Lib:MountingHole_1.5mm_PAD, F.Cu at (164.0, 109.0)
- added H2: MountingHole, Heptachron-Lib:MountingHole_1.5mm_PAD, F.Cu at (164.0, 93.0)
- added H3: MountingHole, Heptachron-Lib:MountingHole_1.5mm_PAD, F.Cu at (132.0, 109.0)
- added H4: MountingHole, Heptachron-Lib:MountingHole_1.5mm_PAD, F.Cu at (132.0, 93.0)
- C4, C7, R13, R14, R15: moved to B.Cu
- moved TP2 65.0 mm to (161.0, 91.5)
- moved TP1 63.0 mm to (158.6, 91.5)
- moved TP6 57.2 mm to (156.6, 107.5)
- moved C4 50.3 mm to (160.2, 95.6)
- moved R16 44.1 mm to (151.9, 91.8)
- moved TP4 43.1 mm to (138.6, 107.3)
- moved C6 42.7 mm to (151.9, 89.8), turned to 180 degrees
- moved R15 41.1 mm to (140.9, 95.7)
- moved C7 37.6 mm to (141.0, 98.5), turned to 180 degrees
- moved R14 29.6 mm to (139.4, 100.0), turned to 180 degrees
- moved R13 29.5 mm to (139.4, 101.7), turned to 180 degrees
- moved J5 1.90 mm to (138.3, 92.1)
- moved J3 1.75 mm to (159.4, 106.8)
- moved J4 1.75 mm to (138.3, 89.6)
- moved J1 0.50 mm to (159.4, 109.5)
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Connections:
- U8 pad 11: unconnected-(U8-PA1-Pad11) -> /LIGHT_IN
- U8 pad 12: unconnected-(U8-PA2-Pad12) -> /LIGHT_EN
- U8 pad 13: /LIGHT_IN -> /RTC_CLK
- U8 pad 2: /LIGHT_EN -> //CE
- U8 pad 6: /RTC_CLK -> unconnected-(U8-PB3-Pad6)
Routing:
- net /SCL: track 0.00 -> 86.2 mm, vias 0 -> 4
- net /CS2: track 0.00 -> 82.3 mm, vias 0 -> 9
- net /CS5: track 0.00 -> 80.4 mm, vias 0 -> 9
- net /SDA: track 0.00 -> 73.9 mm, vias 0 -> 2
- net /BU1: track 0.00 -> 69.2 mm, vias 0 -> 3
- net /CS7: track 0.00 -> 68.0 mm, vias 0 -> 8
- net GND: track 0.00 -> 66.0 mm, vias 0 -> 23
- net /CS6: track 0.00 -> 64.1 mm, vias 0 -> 8
- net +5V: track 0.00 -> 64.0 mm, vias 0 -> 4
- net /CS1: track 0.00 -> 60.3 mm, vias 0 -> 3
- net /CS3: track 0.00 -> 59.1 mm, vias 0 -> 5
- net /CS4: track 0.00 -> 57.1 mm, vias 0 -> 4
- net /SW1: track 0.00 -> 53.2 mm, vias 0 -> 1
- net /RTC_INT: track 0.00 -> 50.4 mm, vias 0 -> 2
- net /RTC_CLK: track 0.00 -> 50.2 mm, vias 0 -> 2
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- added copper zone on F.Cu, net VCC
Other:
- outline, holes or cut-outs redrawn
- board text added: "A. Anderson G. Abrahamsson"
- board text added: "BMS"
- board text added: "Heptachron v0.1 2024"
- board text removed: "BQ25185DLHR"

Commit message: PCB v0.1 [Ordered]
Routing:
- net VCC: track 37.0 -> 108.4 mm, vias 6 -> 18
- net GND: track 66.0 -> 93.4 mm, vias 23 -> 35
- net /LED_EN: track 29.2 -> 30.6 mm
- net /CS2: track 82.3 -> 81.0 mm
- net /BU2: track 49.6 -> 50.7 mm
- net /CS7: track 68.0 -> 68.9 mm
- net /BU1: track 69.2 -> 70.1 mm
- net /CS6: track 64.1 -> 64.8 mm

Commit message: PCB v0.2
Parts:
- C1, C8, C9, IC1, R1, R17, R18, R2, X1: moved to F.Cu
- U1, U2, U3, U4: footprint Heptachron-Lib:7-segment-digit-Cree -> Heptachron-Lib:7-SEGMENT_NEW
- moved C1 28.6 mm to (161.0, 108.3)
- moved R13 28.3 mm to (167.0, 107.7), turned to 90 degrees
- moved R14 28.0 mm to (164.8, 111.9)
- moved TP2 25.3 mm to (135.8, 93.3)
- moved X1 22.5 mm to (157.5, 108.5)
- moved R2 21.2 mm to (153.6, 110.1), turned to 0 degrees
- moved TP6 20.8 mm to (135.8, 106.8)
- moved J1 19.9 mm to (162.2, 89.8)
- moved R1 19.2 mm to (153.6, 112.0), turned to 0 degrees
- moved TP1 18.9 mm to (139.8, 93.3)
- moved J5 14.3 mm to (152.6, 93.6)
- moved J4 14.3 mm to (152.6, 90.6)
- moved R19 11.6 mm to (158.8, 98.0), turned to 90 degrees
- moved IC1 10.3 mm to (158.1, 93.5), turned to 0 degrees
- moved C8 8.66 mm to (152.4, 89.9)
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Connections:
- D37 pad 1: /CS6 -> /CS8
- U7 pad 5: unconnected-(U7-CS8-Pad5) -> /CS8
- U8 pad 2: //CE -> /STAT2
- U8 pad 6: unconnected-(U8-PB3-Pad6) -> /STAT1
Routing:
- net VCC: track 108.4 -> 16.0 mm, vias 18 -> 9
- net GND: track 93.4 -> 31.2 mm, vias 35 -> 23
- net +5V: track 64.0 -> 13.1 mm, vias 4 -> 3
- net /RTC_CLK: track 50.6 -> 12.6 mm, vias 2 -> 3
- net /RTC_INT: track 50.8 -> 15.3 mm, vias 2 -> 1
- net /LED_EN: track 30.6 -> 62.4 mm, vias 2 -> 4
- net //CE: track 27.9 -> 0.00 mm, vias 2 -> 0
- net /CS7: track 68.9 -> 41.1 mm, vias 8 -> 5
- net /STAT2: track 13.5 -> 39.8 mm, vias 1 -> 5
- net /STAT1: track 20.6 -> 38.7 mm, vias 1 -> 3
- net /CS5: track 80.7 -> 63.5 mm, vias 9 -> 8
- net /SCL: track 86.4 -> 70.4 mm, vias 4 -> 6
- net /SDA: track 74.0 -> 58.5 mm, vias 2 -> 3
- net /SW2: track 42.2 -> 28.9 mm, vias 1 -> 3
- net /CS4: track 57.0 -> 44.5 mm, vias 4 -> 1
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- added copper zone on In1.Cu, net GND
- added copper zone on In2.Cu, net VCC
- removed copper zone on B.Cu, net GND
- removed copper zone on F.Cu, net VCC
Other:
- copper layers 2 -> 4
- board text added: "Heptachron v0.2 2024"
- board text removed: "Heptachron v0.1 2024"
