File: PCB/Heptachron/Heptachron.kicad_sch (KiCad schematic)
At the start: 42 parts, among them SW1 SW_Push, SW2 SW_Push, SW3 SW_DP3T, U6 BQ24230RGT, U7 IS31FL3729, U8 ATtiny424-SS, X1 RV-3028-C7

Commit message: Test PCB finished!
Parts:
- removed SW3: SW_DP3T, symbol Switch:SW_DP3T
- added C6, C7: 100n, Capacitor_SMD:C_0603_1608Metric, symbol Device:C_Small
- added J1: Conn_02x03_Counter_Clockwise, Connector_PinHeader_2.54mm:PinHeader_2x03_P2.54mm_Vertical, symbol Connector_Generic:Conn_02x03_Odd_Even
- added Q1: Q_Photo_NPN, LED_SMD:LED_0603_1608Metric, symbol Device:Q_Photo_NPN
- added R16: 10K, Resistor_SMD:R_0603_1608Metric, symbol Device:R_Small
- added SW4: SW_SP3T, Heptachron-Lib:sp3t_jumpers, symbol Switch:SW_SP3T
- C1, C4: footprint (none) -> Capacitor_SMD:C_0603_1608Metric
- C2, C3, C5: footprint (none) -> Capacitor_SMD:C_0805_2012Metric
- R1, R10, R11, R12, R13, R14, R15, R2, R3, R4, R5, R6, R7, R8, R9: footprint (none) -> Resistor_SMD:R_0603_1608Metric
- SW1, SW2: footprint (none) -> Button_Switch_SMD:SW_Push_1P1T_NO_6x6mm_H9.5mm
Connections:
- net +5V: now also J1.4 (Pin_4), SW4.4
- net +BATT: now also J1.2 (Pin_2), SW4.2
- net BMSOUT: now also U6.5 (EN2), SW4.1
- net CHG: no longer U8.2 (PA4)
- net GND: now also C6.2, C7.2, J1.6 (Pin_6), R16.1
- net RX: now also J1.5 (Pin_5)
- net SW1: now also U4.1 (A_A), U4.2 (A_B), U4.3 (A_C), U4.4 (A_D), U4.5 (A_E), U4.6 (A_F), U4.7 (A_G); no longer U1.1 (A_A), U1.2 (A_B), U1.3 (A_C), U1.4 (A_D), U1.5 (A_E), U1.6 (A_F), U1.7 (A_G)
- net SW2: now also U3.1 (A_A), U3.2 (A_B), U3.3 (A_C), U3.4 (A_D), U3.5 (A_E), U3.6 (A_F), U3.7 (A_G); no longer U2.1 (A_A), U2.2 (A_B), U2.3 (A_C), U2.4 (A_D), U2.5 (A_E), U2.6 (A_F), U2.7 (A_G)
- net SW3: now also U2.1 (A_A), U2.2 (A_B), U2.3 (A_C), U2.4 (A_D), U2.5 (A_E), U2.6 (A_F), U2.7 (A_G); no longer U3.1 (A_A), U3.2 (A_B), U3.3 (A_C), U3.4 (A_D), U3.5 (A_E), U3.6 (A_F), U3.7 (A_G)
- net SW4: now also U1.1 (A_A), U1.2 (A_B), U1.3 (A_C), U1.4 (A_D), U1.5 (A_E), U1.6 (A_F), U1.7 (A_G); no longer U4.1 (A_A), U4.2 (A_B), U4.3 (A_C), U4.4 (A_D), U4.5 (A_E), U4.6 (A_F), U4.7 (A_G)
- net TX: now also J1.3 (Pin_3)
- net UPDI: now also J1.1 (Pin_1)
- net VCC: now also C7.1, SW4.3; no longer U6.5 (EN2)
- net LIGHT renamed LIGHT_IN
- net LIGHT_IN: now also C6.1, Q1.2 (E), R16.2
- new net LIGHT_EN: Q1.1 (C), U8.2 (PA4)

Commit message: Add testing PCB [Ordered]
Parts:
- added IC1: BQ25185DLHR, Heptachron-Lib:SON40P220X200X80-11N, symbol Heptachron:BQ25185DLHR
- SW1, SW2: footprint Button_Switch_SMD:SW_Push_1P1T_NO_6x6mm_H9.5mm -> Heptachron-Lib:SW_TL6340AF160Q
Changed lines of the file:
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@@
+    )
+  )
+  (symbol (lib_id "Heptachron:BQ25185DLHR") (at 63.5 73.66 0) (unit 1)
+    (in_bom yes) (on_board yes) (dnp no) (fields_autoplaced)
+    (property "Reference" "IC1" (at 81.28 66.04 0)
+      (effects (font (size 1.27 1.27)))
+    )
+    (property "Value" "BQ25185DLHR" (at 81.28 68.58 0)
+      (effects (font (size 1.27 1.27)))
+    )
+    (property "Footprint" "Heptachron-Lib:SON40P220X200X80-11N" (at 95.25 71.12 0)
+      (effects (font (size 1.27 1.27)) (justify left) hide)
+    )
+    (property "Datasheet" "https://www.ti.com/lit/ds/symlink/bq25185.pdf?ts=1706857561339&ref_url=https%253A%252F%252Fwww.ti.com%252Fproduct%252FBQ25185" (at 95.25 73.66 0)
+      (effects (font (size 1.27 1.27)) (justify left) hide)
+    )
+    (property "Description" "Battery Management NPI  1-CELL 1A STANDALONE LNR HRGR" (at 95.25 76.2 0)
+      (effects (font (size 1.27 1.27)) (justify left) hide)
+    )
+    (property "Height" "0.8" (at 95.25 78.74 0)
+      (effects (font (size 1.27 1.27)) (justify left) hide)
+    )
+    (property "Mouser Part Number" "595-BQ25185DLHR" (at 95.25 81.28 0)
+      (effects (font (size 1.27 1.27)) (justify left) hide)
+    )
+    (property "Mouser Price/Stock" "https://www.mouser.co.uk/ProductDetail/Texas-Instruments/BQ25185DLHR?qs=Z%252BL2brAPG1IbO%2FV3RqsaPw%3D%3D" (at 95.25 83.82 0)
+      (effects (font (size 1.27 1.27)) (justify left) hide)
+    )
+    (property "Manufacturer_Name" "Texas Instruments" (at 95.25 86.36 0)
+      (effects (font (size 1.27 1.27)) (justify left) hide)
+    )
+    (property "Manufacturer_Part_Number" "BQ25185DLHR" (at 95.25 88.9 0)
+      (effects (font (size 1.27 1.27)) (justify left) hide)
+    )
+    (pin "1")
+    (pin "10")
+    (pin "11")
+    (pin "2")
+    (pin "3")
+    (pin "4")
+    (pin "5")
+    (pin "6")
+    (pin "7")
+    (pin "8")
+    (pin "9")
+    (instances
+      (project "Heptachron"
+        (path "/c6ec4407-9aab-4aab-950a-5d337d47ac64"
+          (reference "IC1") (unit 1)
+        )
+      )
     )
   )
@@
       (effects (font (size 1.27 1.27)))
     )
-    (property "Footprint" "Button_Switch_SMD:SW_Push_1P1T_NO_6x6mm_H9.5mm" (at 151.13 115.57 0)
+    (property "Footprint" "Heptachron-Lib:SW_TL6340AF160Q" (at 151.13 115.57 0)
       (effects (font (size 1.27 1.27)) hide)
     )
@@
       (effects (font (size 1.27 1.27)))
     )
-    (property "Footprint" "Button_Switch_SMD:SW_Push_1P1T_NO_6x6mm_H9.5mm" (at 151.13 104.14 0)
-      (effects (font (size 1.27 1.27)) hide)
+    (property "Footprint" "Heptachron-Lib:SW_TL6340AF160Q" (at 151.13 104.14 0)
+      (effects (font (size 1.27 1.27)))
     )
     (property "Datasheet" "~" (at 151.13 104.14 0)

Commit message: Continue PCB
Parts:
- removed J1: Conn_02x03_Counter_Clockwise, Connector_PinHeader_2.54mm:PinHeader_2x03_P2.54mm_Vertical, symbol Connector_Generic:Conn_02x03_Odd_Even
- added D43: ~, LED_SMD:LED_0603_1608Metric, symbol Device:LED_Small
- added J1: GND_MAG, Connector_Wire:SolderWirePad_1x01_SMD_1x2mm, symbol Connector_Generic:Conn_01x01
- added J2: UPDI_MAG, Connector_Wire:SolderWirePad_1x01_SMD_1x2mm, symbol Connector_Generic:Conn_01x01
- added J3: 5V_MAG, Connector_Wire:SolderWirePad_1x01_SMD_1x2mm, symbol Connector_Generic:Conn_01x01
- added J4: BAT+, Connector_Wire:SolderWirePad_1x01_SMD_1x2mm, symbol Connector_Generic:Conn_01x01
- added J5: BAT-, Connector_Wire:SolderWirePad_1x01_SMD_1x2mm, symbol Connector_Generic:Conn_01x01
- added J6: TX, Connector_Wire:SolderWirePad_1x01_SMD_1x2mm, symbol Connector_Generic:Conn_01x01
- added J7: RX, Connector_Wire:SolderWirePad_1x01_SMD_1x2mm, symbol Connector_Generic:Conn_01x01
Connections:
- net +5V: now also J3.1 (Pin_1)
- net +BATT: now also J4.1 (Pin_1)
- net CS6: now also D43.1 (K)
- net GND: now also J1.1 (Pin_1), J5.1 (Pin_1)
- net RX: now also J7.1 (Pin_1)
- net SW5: now also D43.2 (A)
- net TX: now also J6.1 (Pin_1)
- net UPDI: now also J2.1 (Pin_1)
Other:
- note added: "Battery connector"
- note added: "Binary counter SW5 CS 1:6"
- note added: "Colon SW5 CS 6:7"
- note added: "Magnetic connector"
- note added: "TX/RX"
- note removed: "Binary counter CS5 SW 1:5"
- note removed: "Colon CS5 SW 6:7"
- note removed: "Connectors"

Commit message: Continue PCB
Parts:
- removed C2, C3, C5: 4.7u, Capacitor_SMD:C_0805_2012Metric, symbol Device:C_Small
- removed D1: PGD, LED_SMD:LED_0603_1608Metric, symbol Device:LED_Small
- removed D2: CHG, LED_SMD:LED_0603_1608Metric, symbol Device:LED_Small
- removed D3: BAT, LED_SMD:LED_0603_1608Metric, symbol Device:LED_Small
- removed D4: VCC, LED_SMD:LED_0603_1608Metric, symbol Device:LED_Small
- removed J6: TX, Connector_Wire:SolderWirePad_1x01_SMD_1x2mm, symbol Connector_Generic:Conn_01x01
- removed J7: RX, Connector_Wire:SolderWirePad_1x01_SMD_1x2mm, symbol Connector_Generic:Conn_01x01
- removed R10, R11, R12, R9: 1K, Resistor_SMD:R_0603_1608Metric, symbol Device:R_Small
- removed R3, R4, R8: 10K, Resistor_SMD:R_0603_1608Metric, symbol Device:R_Small
- removed R5: 3.3K, Resistor_SMD:R_0603_1608Metric, symbol Device:R_Small
- removed R6: 4.7K, Resistor_SMD:R_0603_1608Metric, symbol Device:R_Small
- removed R7: DNP, Resistor_SMD:R_0603_1608Metric, symbol Device:R_Small
- removed SW4: SW_SP3T, Heptachron-Lib:sp3t_jumpers, symbol Switch:SW_SP3T
- removed U6: BQ24230RGT, Package_DFN_QFN:VQFN-16-1EP_3x3mm_P0.5mm_EP1.68x1.68mm_ThermalVias, symbol Power_Management:BQ24230RGT
- added C10, C8: 1u, Capacitor_SMD:C_0805_2012Metric, symbol Device:C_Small
- added C9: 10u, Capacitor_SMD:C_0805_2012Metric, symbol Device:C_Small
- added R17: 18K, Resistor_SMD:R_0603_1608Metric, symbol Device:R_Small
- added R18: 2K, Resistor_SMD:R_0603_1608Metric, symbol Device:R_Small
- added R19: 10K, Resistor_SMD:R_0603_1608Metric, symbol Device:R_Small
- added TP1: STAT1, TestPoint:TestPoint_Pad_D1.0mm, symbol Connector:TestPoint
- added TP2: STAT2, TestPoint:TestPoint_Pad_D1.0mm, symbol Connector:TestPoint
- added TP3: +5V, TestPoint:TestPoint_Pad_D1.0mm, symbol Connector:TestPoint
- added TP4: VCC, TestPoint:TestPoint_Pad_D1.0mm, symbol Connector:TestPoint
- added TP5: BAT, TestPoint:TestPoint_Pad_D1.0mm, symbol Connector:TestPoint
- added TP6: GND, TestPoint:TestPoint_Pad_D1.0mm, symbol Connector:TestPoint
- J1: renamed from J3; value 5V_MAG -> 5V
- J2: renamed from J1; value GND_MAG -> GND
- J3: renamed from J2; value UPDI_MAG -> UPDI
- Q1: value Q_Photo_NPN -> Q_PH
Connections:
- net PGOOD is gone; now on net RTC_INT: U8.3 (PA5)
- net RX is gone; now on net /CE: U8.12 (PA2)
- net +5V: now also IC1.10 (IN), C8.1, TP3.1
- net +BATT: now also IC1.2 (BAT), C10.2, TP5.1
- net GND: now also IC1.11 (EP), IC1.5 (GND), C10.1, C8.2, C9.1, R17.1, R18.1, R19.1, TP6.1
- net VCC: now also IC1.1 (SYS), C9.2, TP4.1
- net STAT2: now reaches IC1.3 (STAT2)
- net STAT2: now also TP2.1
- net /CE: now reaches IC1.4 (~{CE})
- net at IC1.6 (TS/MR): now also R19.2
- net at IC1.7 (ILIM/VSET): now also R17.2
- net at IC1.8 (ISET): now also R18.2
- net STAT1: now reaches IC1.9 (STAT1)
- net STAT1: now also TP1.1
- net RTC_INT: now reaches X1.2 (INT)
- net TX: no longer names the net of U8.11 (PA1)
- no-connect marks 14 -> 12
Other:
- note added: "Debug pads"
- note removed: "=ITERM"
- note removed: "Debug LEDs"
- note removed: "R_ISET = 870/I_CHG R_ILIM = 1530/I_MAX"
- note removed: "System power switch"
- note removed: "TX/RX"
- moved on the sheet: IC1, J1, J2, J3, J4, J5, SW1, SW2

Commit message: Continue PCB
Parts:
- removed TP3: +5V, TestPoint:TestPoint_Pad_D1.0mm, symbol Connector:TestPoint
- removed TP5: BAT, TestPoint:TestPoint_Pad_D1.0mm, symbol Connector:TestPoint
- added H1, H2, H3, H4: MountingHole, Heptachron-Lib:MountingHole_1.5mm_PAD, symbol Mechanical:MountingHole
Connections:
- net LIGHT_EN: now also U8.12 (PA2); no longer U8.2 (PA4)
- net LIGHT_IN: now also U8.11 (PA1); no longer U8.13 (PA3)
- net RTC_CLK: now also U8.13 (PA3); no longer U8.6 (PB3)
- net /CE: now also U8.2 (PA4); no longer U8.12 (PA2)
Other:
- note added: "Mounting holes"
- moved on the sheet: D43, J1, J2, J3, J4, J5, TP1, TP2, TP4, TP6

Commit message: PCB v0.2
Parts:
- U1, U2, U3, U4: footprint Heptachron-Lib:7-segment-digit-Cree -> Heptachron-Lib:7-SEGMENT_NEW
Connections:
- net CS6: no longer D37.1 (K)
- net STAT1: now also U8.6 (PB3)
- net STAT2: now also U8.2 (PA4)
- net /CE: no longer U8.2 (PA4)
- net CS8: now reaches U7.5 (CS8)
- net CS8: now also D37.1 (K)
- no-connect marks 12 -> 11
Other:
- note added: "Colon SW5 CS 7:8"
- note added: "Digit 1 SW4 CS 1:7 ─── │ │ │ │ ─── │ │ │ │ ───"
- note added: "Digit 2 SW3 CS 1:7 ─── │ │ │ │ ─── │ │ │ │ ───"
- note added: "Digit 3 SW2 CS 1:7 ─── │ │ │ │ ─── │ │ │ │ ───"
- note added: "Digit 4 SW1 CS 1:7 ─── │ │ │ │ ─── │ │ │ │ ───"
- note added: "│ │ │ │ │ │"
- note added: "◄ A F ▲ ▼ B ◄ G E ▲ ▼ C ◄ D"
- note removed: "CS:n - Current sink 'n', one for each digit [CATHODE] SW:n - Switch power source, one for each segment [ANODE] SW1: A, SW2: B, ..., SW7: G ◄ A F ▲ ▼ B ◄ G E ▲ ▼ C ◄ D"
- note removed: "Colon SW5 CS 6:7"
- note removed: "Digit 1 CS1 SW 1:7 ─── │ │ │ │ ─── │ │ │ │ ───"
- note removed: "Digit 2 CS2 SW 1:7 ─── │ │ │ │ ─── │ │ │ │ ───"
- note removed: "Digit 3 CS3 SW 1:7 ─── │ │ │ │ ─── │ │ │ │ ───"
- note removed: "Digit 4 CS4 SW 1:7 ─── │ │ │ │ ─── │ │ │ │ ───"
- note removed: "│ │ │ │ │"
Changed lines of the file:
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@@
   (no_connect (at 121.92 67.31))
   (no_connect (at 121.92 64.77))
-  (no_connect (at 121.92 54.61))
   (no_connect (at 121.92 72.39))
   (no_connect (at 121.92 59.69))
@@
     (stroke (width 0) (type default))
   )
+  (wire (pts (xy 40.64 132.08) (xy 41.91 132.08))
+    (stroke (width 0) (type default))
+  )
   (wire (pts (xy 224.79 200.66) (xy 227.33 200.66))
     (stroke (width 0) (type default))
@@
     (stroke (width 0) (type default))
   )
-  (text "Digit 3\n       \nCS3    \nSW 1:7 \n       \n  ───  \n│     │\n│     │\n  ───  \n│     │\n│     │\n  ───  "
+  (text "Digit 3\n       \nSW2    \nCS 1:7  \n       \n  ───  \n│     │\n│     │\n  ───  \n│     │\n│     │\n  ───  "
     (at 317.5 59.69 0)
     (effects (font (size 2 2) italic) (justify left bottom))
@@
     (effects (font (size 2 2)) (justify left bottom))
   )
-  (text "Digit 2\n       \nCS2    \nSW 1:7 \n       \n  ───  \n│     │\n│     │\n  ───  \n│     │\n│     │\n  ───  "
+  (text "Digit 2\n       \nSW3    \nCS 1:7 \n       \n  ───  \n│     │\n│     │\n  ───  \n│     │\n│     │\n  ───  "
     (at 252.73 59.69 0)
     (effects (font (size 2 2) italic) (justify left bottom))
   )
-  (text "CS:n  -   Current sink 'n', one for each digit       [CATHODE]\n                                                              \nSW:n  -   Switch power source, one for each segment  [ANODE]  \n               SW1: A, SW2: B, ..., SW7: G                    \n                                                                                            \n                                                              \n                           ◄ A                                \n                                                              \n                                                              \n                     F              ▲                         \n                                                              \n                     ▼              B                         \n                                                              \n                           ◄ G                                \n                                                              \n                     E              ▲                         \n                                                              \n                     ▼              C                         \n                                                              \n                                                              \n                           ◄ D                                "
-    (at 184.15 154.94 0)
+  (text "                 \n                                                                                            \n                                                              \n                           ◄ A                                \n                                                              \n                                                              \n                     F              ▲                         \n                                                              \n                     ▼              B                         \n                                                              \n                           ◄ G                                \n                                                              \n                     E              ▲                         \n                                                              \n                     ▼              C                         \n                                                              \n                                                              \n                           ◄ D                                "
+    (at 191.77 146.05 0)
     (effects (font (size 1.27 1.27)) (justify left bottom))
   )
@@
     (effects (font (size 2 2)) (justify left bottom))
   )
-  (text "│  │  │  │  │" (at 283.21 67.31 0)
+  (text "│  │  │  │  │  │" (at 281.94 67.31 0)
     (effects (font (size 1.27 1.27)) (justify left bottom))
   )
@@
     (effects (font (size 1.27 1.27)) (justify left bottom))
   )
-  (text "Colon\n\nSW5\nCS 6:7" (at 270.51 118.11 0)
+  (text "Colon\n\nSW5\nCS 7:8" (at 270.51 118.11 0)
     (effects (font (size 1.27 1.27) italic) (justify left bottom))
   )
@@
     (effects (font (size 2 2)) (justify left bottom))
   )
-  (text "Digit 1\n       \nCS1    \nSW 1:7 \n       \n  ───  \n│     │\n│     │\n  ───  \n│     │\n│     │\n  ───  "
+  (text "Digit 1\n       \nSW4    \nCS 1:7 \n       \n  ───  \n│     │\n│     │\n  ───  \n│     │\n│     │\n  ───  "
     (at 213.36 59.69 0)
     (effects (font (size 2 2) italic) (justify left bottom))
@@
     (effects (font (size 2 2)) (justify left bottom))
   )
-  (text "Digit 4\n       \nCS4    \nSW 1:7 \n       \n  ───  \n│     │\n│     │\n  ───  \n│     │\n│     │\n  ───  "
+  (text "Digit 4\n       \nSW1    \nCS 1:7 \n       \n  ───  \n│     │\n│     │\n  ───  \n│     │\n│     │\n  ───  "
     (at 356.87 59.69 0)
     (effects (font (size 2 2) italic) (justify left bottom))
@@
     (effects (font (size 1.27 1.27)) (justify left bottom))
   )
-  (label "{slash}CE" (at 77.47 134.62 0) (fields_autoplaced)
-    (effects (font (size 1.27 1.27)) (justify left bottom))
-  )
   (label "STAT1" (at 81.28 50.8 180) (fields_autoplaced)
     (effects (font (size 1.27 1.27)) (justify right bottom))
   )
+  (label "STAT2" (at 77.47 134.62 0) (fields_autoplaced)
+    (effects (font (size 1.27 1.27)) (justify left bottom))
+  )
   (label "STAT2" (at 35.56 53.34 180) (fields_autoplaced)
     (effects (font (size 1.27 1.27)) (justify right bottom))
@@
     (effects (font (size 1.27 1.27)) (justify left bottom))
   )
-  (label "CS6" (at 274.32 148.59 90) (fields_autoplaced)
+  (label "CS8" (at 274.32 148.59 90) (fields_autoplaced)
     (effects (font (size 1.27 1.27)) (justify left bottom))
   )
@@
   (label "CS2" (at 231.14 87.63 0) (fields_autoplaced)
     (effects (font (size 1.27 1.27)) (justify left bottom))
+  )
+  (label "CS8" (at 121.92 54.61 180) (fields_autoplaced)
+    (effects (font (size 1.27 1.27)) (justify right bottom))
   )
   (label "CS1" (at 270.51 85.09 0) (fields_autoplaced)
@@
     (effects (font (size 1.27 1.27)) (justify left bottom))
   )
+  (label "STAT1" (at 40.64 132.08 180) (fields_autoplaced)
+    (effects (font (size 1.27 1.27)) (justify right bottom))
+  )
   (label "CS2" (at 270.51 87.63 0) (fields_autoplaced)
     (effects (font (size 1.27 1.27)) (justify left bottom))
@@
     (effects (font (size 1.27 1.27)) (justify left bottom))
   )
-  (label "CS1" (at 335.28 85.09 0) (fields_autoplaced)
-    (effects (font (size 1.27 1.27)) (justify left bottom))
-  )
   (label "CS7" (at 121.92 52.07 180) (fields_autoplaced)
     (effects (font (size 1.27 1.27)) (justify right bottom))
   )
+  (label "CS1" (at 335.28 85.09 0) (fields_autoplaced)
+    (effects (font (size 1.27 1.27)) (justify left bottom))
+  )
   (label "CS1" (at 121.92 36.83 180) (fields_autoplaced)
     (effects (font (size 1.27 1.27)) (justify right bottom))
@@
       (effects (font (size 1.27 1.27)))
     )
-    (property "Footprint" "Heptachron-Lib:7-segment-digit-Cree" (at 259.08 93.98 0)
+    (property "Footprint" "Heptachron-Lib:7-SEGMENT_NEW" (at 259.08 93.98 0)
       (effects (font (size 1.27 1.27)) hide)
     )
@@
       (effects (font (size 1.27 1.27)))
     )
-    (property "Footprint" "Heptachron-Lib:7-segment-digit-Cree" (at 363.22 93.98 0)
+    (property "Footprint" "Heptachron-Lib:7-SEGMENT_NEW" (at 363.22 93.98 0)
       (effects (font (size 1.27 1.27)) hide)
     )
@@
       (effects (font (size 1.27 1.27)))
     )
-    (property "Footprint" "Heptachron-Lib:7-segment-digit-Cree" (at 219.71 93.98 0)
+    (property "Footprint" "Heptachron-Lib:7-SEGMENT_NEW" (at 219.71 93.98 0)
       (effects (font (size 1.27 1.27)) hide)
     )
@@
       (effects (font (size 1.27 1.27)))
     )
-    (property "Footprint" "Heptachron-Lib:7-segment-digit-Cree" (at 323.85 93.98 0)
-      (effects (font (size 1.27 1.27)) hide)
-    )
+    (property "Footprint" "Heptachron-Lib:7-SEGMENT_NEW" (at 323.85 93.98 0)
+      (effects (font (size 1.27 1.27)) hide)
+    )
